File: HW/Proto/rbServoProto.kicad_pcb (KiCad board)
At the start: 2 copper layers, 50 x 27 mm, 30 parts, among them IC1 ATMEGA32M1_QFN32, P1 EXTCON, P2 POT, P3 MOTOR, Q1 PMF170XP, U1 TJA1050, U2 LM3480, U3 DRV8837-DSG, X1 16MHz

Commit message: Work on all fronts. The software is taking shape now.
Parts:
- removed C1, C10, C11, C6, C7, C8: 100n, SMD-0805
- removed C2, C3: 0µ1, SMD-0805
- removed C4: 12p, SMD-0805
- removed C5: 10p, SMD-0805
- removed C9: cCAN, SMD-0805
- removed D1, D2: LED, SMD-0805-LED
- removed IC1: ATMEGA32M1_QFN32, TQFP-32
- removed ISP1: ATMEL_ISP-6P, DIN_41651_3x2
- removed P1: EXTCON, MPT_0,5/2,54x04
- removed P2: POT, MPT_0,5/2,54x03
- removed P3: MOTOR, MPT_0,5/2,54x02
- removed Q1: PMF170XP, SC70-3
- removed R1: 12k, SMD-0805
- removed R2: 22k, SMD-0805
- removed R3, R4: 400, SMD-0805
- removed R5: 10k, SMD-0805
- removed R6, R7: rCAN, SMD-0805
- removed U1: TJA1050, SOIC-8
- removed U2: LM3480, SOT-23_TO-236AB
- removed U3: DRV8837-DSG, SMD-PWSON-8
- removed X1: 16MHz, XTAL_SMD_2mm5x2mm
- added C201: 100n, SMD_Discrete:0402-1005, F.Cu at (162.9, 117.4)
- added C202: 0µ1, SMD_Discrete:0402-1005, F.Cu at (157.1, 99.0)
- added C203: 0µ1, SMD_Discrete:0402-1005, F.Cu at (153.8, 105.5)
- added C204: 12p, SMD_Discrete:0402-1005, F.Cu at (167.5, 112.3)
- added C205: 12p, SMD_Discrete:0402-1005, F.Cu at (168.5, 112.3)
- added C206: 100n, SMD_Discrete:0402-1005, F.Cu at (158.0, 105.4)
- added C207: 100n, SMD_Discrete:0402-1005, F.Cu at (160.0, 105.4)
- added C208: 100n, SMD_Discrete:0402-1005, F.Cu at (159.0, 114.6)
- added C209: cCAN, SMD_Discrete:0402-1005, F.Cu at (156.8, 118.4)
- added C210: 10u, SMD_Tantalum:A-3216-18, F.Cu at (157.1, 102.0)
- added C211: 100n, SMD_Discrete:0402-1005, F.Cu at (158.8, 103.5)
- added C212: 2u2, SMD_Discrete:0402-1005, F.Cu at (165.4, 103.5)
- added D201: LED, SMD_Discrete:LED-0402-1005, F.Cu at (163.9, 115.5)
- added D202: LED, SMD_Discrete:LED-0402-1005, F.Cu at (164.9, 115.5)
- added IC201: ATMEGA32M1_QFN32, QFN:QFN-32_0mm65, F.Cu at (159.0, 110.0)
- added ISP101: ATMEL_ISP-6P, Pin_Header_1.27mm:2x3-RECEPTACLE-SMD, F.Cu at (167.4, 107.4)
- added OL101: OUTLINE, Outlines:rbServo_Outline, F.Cu at (161.0, 111.6)
- added P101: EXTCON, rbv_connectors:MPT_0,5%2f2,54x04, B.Cu at (161.3, 122.2)
- added P104: p5V, Vias_and_Pads:0.7x1.5mm, F.Cu at (162.2, 105.6)
- added P105: pGND, Vias_and_Pads:0.7x1.5mm, F.Cu at (164.2, 105.6)
- added P109: pA, Vias_and_Pads:0.7x1.5mm, F.Cu at (164.2, 107.6)
- added P113: M+, Vias_and_Pads:0.7x1.5mm, F.Cu at (164.2, 98.3)
- added P114: M-, Vias_and_Pads:0.7x1.5mm, F.Cu at (162.1, 98.3)
- added Q201: PMF170XP, SOT:SOT323_SC-70, F.Cu at (154.4, 99.9)
- added R201: 12k, SMD_Discrete:0402-1005, F.Cu at (153.5, 108.5)
- added R202: 22k, SMD_Discrete:0402-1005, F.Cu at (153.5, 109.5)
- added R203: 400, SMD_Discrete:0402-1005, F.Cu at (163.9, 117.4)
- added R204: 400, SMD_Discrete:0402-1005, F.Cu at (164.9, 117.4)
- added R205: 10k, SMD_Discrete:0402-1005, F.Cu at (153.5, 110.5)
- added R206: rCAN, SMD_Discrete:0402-1005, F.Cu at (156.8, 117.4)
- added R207: rCAN, SMD_Discrete:0402-1005, F.Cu at (156.8, 116.4)
- added R208: 4k7, SMD_Discrete:0402-1005, F.Cu at (153.5, 111.5)
- added R209: 200m, SMD_Discrete:0805-2012, F.Cu at (165.9, 100.4)
- added U201: TJA1051, SOT:SOT782-1, F.Cu at (160.1, 117.4)
- added U202: LM3480, SOT:SOT-23, F.Cu at (154.2, 103.2)
- added U203: DRV8833-QFN, QFN:PQFN-16, F.Cu at (162.1, 101.7)
- added X201: 16MHz, XTAL:SMD-2.5x2mm, F.Cu at (165.0, 112.3)
Routing:
- net +5V: track 93.3 -> 15.9 mm, vias 5 -> 1
- net GND: track 78.3 -> 15.2 mm, vias 10 -> 6
- net /Core/Isense: track 0.00 -> 23.2 mm, vias 0 -> 4
- net /Core/ISP_MOSI: track 22.4 -> 0.00 mm
- net /Core/ISP_SCK: track 19.3 -> 0.00 mm
- net N-000041: track 18.9 -> 0.00 mm
- net /Core/CAN_RX: track 15.3 -> 0.00 mm
- net /Core/PWM_A: track 0.00 -> 13.5 mm, vias 0 -> 2
- net N-000014: track 12.7 -> 0.00 mm
- net /Core/aPot: track 13.6 -> 1.86 mm
- net /Core/ISP_RES: track 14.1 -> 2.50 mm, vias 0 -> 1
- net /Core/ledA: track 13.9 -> 3.65 mm
- net /Core/F_PWM: track 9.68 -> 0.00 mm
- net /Core/R_PWM: track 9.55 -> 0.00 mm
- net /Core/CAN_TX: track 9.03 -> 0.00 mm
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- added copper zone on Inner2.Cu, net /Core/Isense
- added copper zone on B.Cu, net /Core/M+
- added copper zone on F.Cu, net /Core/M+
- added copper zone on F.Cu, net /Core/M-
- added copper zone on Inner1.Cu, net /Core/uIn
- removed copper zone on B.Cu, net +BATT
- removed copper zone on F.Cu, net +BATT
- removed copper zone on B.Cu, net /Core/uIn
- removed copper zone on F.Cu, net /Core/uIn
- removed copper zone on B.Cu, net GND
- removed copper zone on F.Cu, net GND
Other:
- board size 50 x 27 mm -> 19 x 32 mm
- copper layers 2 -> 4
- net class Default: clearance 0.1524 -> 0.127; trace_width 0.28 -> 0.127; via_dia 0.6858 -> 0.4572; via_drill 0.3302 -> 0.254
- net class Power: clearance 0.2 -> 0.127; trace_width 0.55 -> 0.35; via_dia 0.6858 -> 0.4572; via_drill 0.3302 -> 0.254
- net class Supply removed
- rule pad_to_mask_clearance: 0.2 -> 0.07
- rule trace_clearance: 0.1524 -> 0.127
- rule trace_min: 0.1524 -> 0.127
- rule via_min_drill: 0.3302 -> 0.254
- rule via_min_size: 0.6858 -> 0.4572
- board text removed: "+"
- board text removed: "+5V"
- board text removed: "-"
- board text removed: "BATT+"
- board text removed: "CAN_H"
- board text removed: "CAN_L"
- board text removed: "GND"
- board text removed: "POT"
- board text removed: "Rev B"
