File: HW/Proto/rbServoProto.sch (KiCad schematic (older format))
At the start: 4 parts, among them P1 EXTCON, P2 POT, P3 MOTOR

Commit message: Work on all fronts. The software is taking shape now.
Parts:
- removed P2: POT, symbol CONN_3
- removed P3: MOTOR, symbol CONN_2
- added OL101: OUTLINE, symbol LOGO
- added P104: p5V, symbol CONN_1
- added P105: pGND, symbol CONN_1
- added P109: pA, symbol CONN_1
- added P113: M+, symbol CONN_1
- added P114: M-, symbol CONN_1
- renumbered ISP1 to ISP101, P1 to P101
Connections:
- net +5V: now also P104.1
- net CAN_HIGH: now also P101.2 (P2); no longer P101.3 (P3)
- net CAN_LOW: now also P101.3 (P3); no longer P101.2 (P2)
- net GND: now also P101.1 (P1), P105.1; no longer P101.4 (P4)
- net MOTOR+: now also P113.1
- net MOTOR-: now also P114.1
- net aPOT: now also P109.1
- net uIn: now also P101.4 (P4); no longer P101.1 (P1)
Changed lines of the file:
@@
 EESchema Schematic File Version 2
+LIBS:rbv_interface
+LIBS:rbv_mosfet
+LIBS:rbv_pcb_extras
+LIBS:rbv_linear
+LIBS:rbv_mcu
+LIBS:rbv_regul
+LIBS:rbv_connectors
+LIBS:rbv_device
+LIBS:rbv_drivers
 LIBS:power
 LIBS:device
@@
 LIBS:contrib
 LIBS:valves
-LIBS:rbv_connectors
-LIBS:rbv_device
-LIBS:rbv_drivers
-LIBS:rbv_mcu
-LIBS:rbv_linear
-LIBS:rbv_regul
-LIBS:rbv_interface
-LIBS:rbv_mosfet
-LIBS:rbv_pcb_extras
+LIBS:rbServoProto-cache
 EELAYER 24 0
 EELAYER END
@@
 $EndDescr
 $Comp
-L CONN_4 P1
+L CONN_4 P101
 U 1 1 4F2DC381
 P 3800 3550
-F 0 "P1" V 3750 3550 50  0000 C CNN
+F 0 "P101" V 3750 3550 50  0000 C CNN
 F 1 "EXTCON" V 3850 3550 50  0000 C CNN
 F 2 "" H 3800 3550 60  0001 C CNN
 F 3 "" H 3800 3550 60  0001 C CNN
 	1    3800 3550
-	-1   0    0    -1
+	-1   0    0    1
 $EndComp
 Text Label 7300 4400 2    60   ~ 0
@@
 L +5V #PWR01
 U 1 1 4E74CD8D
-P 4300 4200
-F 0 "#PWR01" H 4300 4290 20  0001 C CNN
-F 1 "+5V" H 4300 4290 30  0000 C CNN
-F 2 "" H 4300 4200 60  0001 C CNN
-F 3 "" H 4300 4200 60  0001 C CNN
-	1    4300 4200
+P 4650 4200
+F 0 "#PWR01" H 4650 4290 20  0001 C CNN
+F 1 "+5V" H 4650 4290 30  0000 C CNN
+F 2 "" H 4650 4200 60  0001 C CNN
+F 3 "" H 4650 4200 60  0001 C CNN
+	1    4650 4200
 	1    0    0    -1
 $EndComp
@@
 Text Label 4650 3600 2    60   ~ 0
 CAN_HIGH
-Text Label 4800 2600 0    60   ~ 0
+Text Label 4750 2600 0    60   ~ 0
 ISP_RES
-Text Label 4800 2400 0    60   ~ 0
+Text Label 4750 2400 0    60   ~ 0
 ISP_MISO
-Text Label 4800 2500 0    60   ~ 0
+Text Label 4750 2500 0    60   ~ 0
 ISP_SCK
-Text Label 6900 2500 2    60   ~ 0
+Text Label 6950 2500 2    60   ~ 0
 ISP_MOSI
 $Comp
@@
 	4150 3400 5050 3400
 Wire Wire Line
-	4300 4200 4300 4650
+	4650 4200 4650 4450
 Wire Wire Line
 	6600 2800 6600 2600
 Wire Wire Line
-	6600 2600 6450 2600
-Wire Wire Line
 	6600 2250 6600 2400
 Wire Wire Line
-	6600 2400 6450 2400
-Wire Wire Line
-	6900 2500 6450 2500
-Wire Wire Line
-	5250 2500 4800 2500
-Wire Wire Line
-	5250 2400 4800 2400
-Wire Wire Line
-	5250 2600 4800 2600
+	6450 2500 6950 2500
+Wire Wire Line
+	5250 2500 4750 2500
+Wire Wire Line
+	5250 2400 4750 2400
+Wire Wire Line
+	5250 2600 4750 2600
 Wire Wire Line
 	4150 3600 5050 3600
 Wire Wire Line
-	6750 4400 7500 4400
-Wire Wire Line
 	6750 4600 7500 4600
 Wire Wire Line
@@
 Wire Wire Line
 	4150 3500 5050 3500
-Text Label 4650 4550 2    60   ~ 0
+Text Label 4600 4550 2    60   ~ 0
 aPOT
 Wire Wire Line
-	5050 4550 4150 4550
+	4150 4550 5050 4550
 $Sheet
 S 5050 3050 1700 2050
@@
 F0 "Core" 50
 F1 "../common/rbServoCore.sch" 50
-F2 "MOTOR+" O R 6750 4400 60
-F3 "MOTOR-" O R 6750 4600 60
+F2 "M+" O R 6750 4400 60
+F3 "M-" O R 6750 4600 60
 F4 "aPot" I L 5050 4550 60
 F5 "ISP_MISO" O R 6750 3650 60
@@
 	7250 3650 6750 3650
 $Comp
-L ATMEL_ISP-6P ISP1
+L ATMEL_ISP-6P ISP101
 U 1 1 50B6476E
 P 5850 2500
-F 0 "ISP1" H 5650 2800 60  0000 C CNN
+F 0 "ISP101" H 5650 2800 60  0000 C CNN
 F 1 "ATMEL_ISP-6P" H 5850 2200 60  0000 C CNN
 F 2 "" H 5850 2500 60  0001 C CNN
@@
 	1    0    0    -1
 $EndComp
-$Comp
-L CONN_3 P2
-U 1 1 50B64948
-P 3800 4650
-F 0 "P2" V 3750 4650 50  0000 C CNN
-F 1 "POT" V 3850 4650 40  0000 C CNN
-F 2 "" H 3800 4650 60  0001 C CNN
-F 3 "" H 3800 4650 60  0001 C CNN
-	1    3800 4650
-	-1   0    0    -1
-$EndComp
-$Comp
-L CONN_2 P3
-U 1 1 50B64B0C
-P 7850 4500
-F 0 "P3" V 7800 4500 40  0000 C CNN
-F 1 "MOTOR" V 7900 4500 40  0000 C CNN
-F 2 "" H 7850 4500 60  0001 C CNN
-F 3 "" H 7850 4500 60  0001 C CNN
-	1    7850 4500
-	1    0    0    -1
-$EndComp
 Text Label 4650 3400 2    60   ~ 0
 uIn
@@
 L GND #PWR05
 U 1 1 50B6786D
-P 4650 5000
-F 0 "#PWR05" H 4650 5000 30  0001 C CNN
-F 1 "GND" H 4650 4930 30  0001 C CNN
-F 2 "" H 4650 5000 60  0001 C CNN
-F 3 "" H 4650 5000 60  0001 C CNN
-	1    4650 5000
-	1    0    0    -1
-$EndComp
-Text Label 4650 4750 2    60   ~ 0
+P 4650 4900
+F 0 "#PWR05" H 4650 4900 30  0001 C CNN
+F 1 "GND" H 4650 4830 30  0001 C CNN
+F 2 "" H 4650 4900 60  0001 C CNN
+F 3 "" H 4650 4900 60  0001 C CNN
+	1    4650 4900
+	1    0    0    -1
+$EndComp
+Text Label 4600 4650 2    60   ~ 0
 GND
 Wire Wire Line
-	4150 4750 4650 4750
-Wire Wire Line
-	4650 4750 4650 5000
-Wire Wire Line
-	4300 4650 4150 4650
+	4150 4650 4650 4650
+Wire Wire Line
+	4650 4650 4650 4900
+Wire Wire Line
+	4650 4450 4150 4450
+$Comp
+L CONN_1 P113
+U 1 1 53165F78
+P 7650 4400
+F 0 "P113" H 7730 4400 40  0000 L CNN
+F 1 "M+" H 7650 4455 30  0001 C CNN
+F 2 "" H 7650 4400 60  0000 C CNN
+F 3 "" H 7650 4400 60  0000 C CNN
+	1    7650 4400
+	1    0    0    -1
+$EndComp
+$Comp
+L CONN_1 P114
+U 1 1 53165F8C
+P 7650 4600
+F 0 "P114" H 7730 4600 40  0000 L CNN
+F 1 "M-" H 7650 4655 30  0001 C CNN
+F 2 "" H 7650 4600 60  0000 C CNN
+F 3 "" H 7650 4600 60  0000 C CNN
+	1    7650 4600
+	1    0    0    -1
+$EndComp
+$Comp
+L CONN_1 P104
+U 1 1 531660F0
+P 4000 4450
+F 0 "P104" H 4080 4450 40  0000 L CNN
+F 1 "p5V" H 4000 4505 30  0001 C CNN
+F 2 "" H 4000 4450 60  0000 C CNN
+F 3 "" H 4000 4450 60  0000 C CNN
+	1    4000 4450
+	-1   0    0    1
+$EndComp
+$Comp
+L CONN_1 P105
+U 1 1 53166127
+P 4000 4650
+F 0 "P105" H 4080 4650 40  0000 L CNN
+F 1 "pGND" H 4000 4705 30  0001 C CNN
+F 2 "" H 4000 4650 60  0000 C CNN
+F 3 "" H 4000 4650 60  0000 C CNN
+	1    4000 4650
+	-1   0    0    1
+$EndComp
+$Comp
+L CONN_1 P109
+U 1 1 5316615E
+P 4000 4550
+F 0 "P109" H 4080 4550 40  0000 L CNN
+F 1 "pA" H 4000 4605 30  0001 C CNN
+F 2 "" H 4000 4550 60  0000 C CNN
+F 3 "" H 4000 4550 60  0000 C CNN
+	1    4000 4550
+	-1   0    0    1
+$EndComp
+Wire Wire Line
+	6600 2600 6450 2600
+Wire Wire Line
+	6600 2400 6450 2400
+Wire Wire Line
+	7500 4400 6750 4400
+$Comp
+L LOGO OL101
+U 1 1 5318F271
+P 10750 6250
+F 0 "OL101" H 10750 6200 60  0000 C CNN
+F 1 "OUTLINE" H 10750 6300 60  0000 C CNN
+F 2 "" H 10750 6250 60  0000 C CNN
+F 3 "" H 10750 6250 60  0000 C CNN
+	1    10750 6250
+	1    0    0    -1
+$EndComp
 $EndSCHEMATC
