File: HW/rbServoCore.sch (KiCad schematic (older format))
At the start: 29 parts, among them IC201 ATMEGA32M1_QFN32, Q201 PMF170XP, U201 TJA1051, U202 LM3480, U203 DRV8833-QFN, X201 16MHz

Commit message: -Swapped CAN_H and CAN_L -Changed a few labels - All new layout that should fit i a servo
Signed-off-by: RasmusB <RasmusB@users.noreply.github.com>
Connections:
- net GND: now also D201.2 (K), D202.2 (K); no longer R203.2, R204.2
- net Isense: now also IC201.17 (PC4(ADC8)); no longer IC201.26 (PB5(ADC6))
- net aPot: now also IC201.26 (PB5(ADC6)); no longer IC201.16 (PB2(ADC5))
- net ledA: now also IC201.18 (PC5(ADC9)), R203.1; no longer D201.1 (A), IC201.8 (PB0(MISO))
- net ledB: now also IC201.22 (PC6(ADC10)), R204.1; no longer D202.1 (A), IC201.9 (PB1(MOSI))
- net m_EN: now also IC201.16 (PB2(ADC5)); no longer IC201.15 (PD7)
- net m_FAULT: now also IC201.15 (PD7)
- net uBattFB: now also IC201.13 (PD5(ADC2)); no longer IC201.27 (PB6(ADC7))
- net vInt: now reaches C212.1, U203.12 (VINT)
- new net: D201.1 (A), R203.2
- new net: D202.1 (A), R204.2
- no-connect marks 10 -> 5
Other:
- moved on the sheet: D201, D202, R203, R204
Changed lines of the file:
@@
 	1    0    0    -1
 $EndComp
-Text Label 6900 4750 2    60   ~ 0
+Text Label 6950 4750 2    60   ~ 0
 ISP_SCK
-Text Label 6900 4550 2    60   ~ 0
+Text Label 6950 4550 2    60   ~ 0
 ISP_MISO
 Text Label 3500 2750 0    60   ~ 0
 ISP_RES
-Text Label 6900 4650 2    60   ~ 0
+Text Label 6950 4650 2    60   ~ 0
 ISP_MOSI
 $Comp
@@
 Text Label 7800 3300 0    60   ~ 0
 m_EN
-Text Label 6800 5050 2    60   ~ 0
+Text Label 6800 2750 2    60   ~ 0
 m_EN
 $Comp
@@
 Text Label 1600 3850 2    60   ~ 0
 uBattFB
-Text Label 6900 3150 2    60   ~ 0
+Text Label 6900 4850 2    60   ~ 0
 uBattFB
 $Comp
 L LED D201
 U 1 1 50B64426
-P 2000 3500
-F 0 "D201" H 2000 3600 50  0000 C CNN
-F 1 "LED" H 2000 3400 50  0000 C CNN
-F 2 "" H 2000 3500 60  0001 C CNN
-F 3 "" H 2000 3500 60  0001 C CNN
-	1    2000 3500
+P 2000 4200
+F 0 "D201" H 2000 4300 50  0000 C CNN
+F 1 "LED" H 2000 4100 50  0000 C CNN
+F 2 "" H 2000 4200 60  0001 C CNN
+F 3 "" H 2000 4200 60  0001 C CNN
+	1    2000 4200
 	0    -1   1    0
 $EndComp
 Text Label 2000 3000 3    60   ~ 0
 ledA
-Text Label 6900 2550 2    60   ~ 0
+Text Label 6900 3950 2    60   ~ 0
 ledA
 Wire Wire Line
 	9200 5250 9200 5000
 Wire Wire Line
-	6350 4550 6900 4550
+	6350 4550 6950 4550
 Connection ~ 4000 3650
 Wire Wire Line
@@
 	1900 6950 1350 6950
 Wire Wire Line
-	6900 5050 6350 5050
+	6900 2750 6350 2750
 Wire Wire Line
 	3500 2750 4450 2750
@@
 	3700 4200 3700 4350
 Wire Wire Line
-	6900 4650 6350 4650
+	6950 4650 6350 4650
 Wire Wire Line
 	3150 1250 3300 1250
@@
 	4000 1950 4000 2100
 Wire Wire Line
-	8400 3650 7800 3650
+	7800 3650 8400 3650
 Wire Wire Line
 	7800 3550 8400 3550
@@
 Connection ~ 3150 3650
 Wire Wire Line
-	6350 4750 6900 4750
+	6350 4750 6950 4750
 Wire Wire Line
 	10000 3500 10650 3500
@@
 Connection ~ 1150 3850
 Wire Wire Line
-	6900 3150 6350 3150
-Wire Wire Line
-	6350 2550 6900 2550
+	6900 4850 6350 4850
+Wire Wire Line
+	6350 3950 6900 3950
 $Comp
 L C C211
@@
 	1    0    0    -1
 $EndComp
-Text Label 6900 2750 2    60   ~ 0
+Text Label 6900 3050 2    60   ~ 0
 aPOT
 Wire Wire Line
-	6900 2750 6350 2750
-Text Label 6900 2650 2    60   ~ 0
+	6900 3050 6350 3050
+Text Label 6900 4050 2    60   ~ 0
 ledB
 Wire Wire Line
-	6350 2650 6900 2650
+	6350 4050 6900 4050
 Text Label 2400 3000 3    60   ~ 0
 ledB
@@
 L LED D202
 U 1 1 50B644D4
-P 2400 3500
-F 0 "D202" H 2400 3600 50  0000 C CNN
-F 1 "LED" H 2400 3400 50  0000 C CNN
-F 2 "" H 2400 3500 60  0001 C CNN
-F 3 "" H 2400 3500 60  0001 C CNN
-	1    2400 3500
+P 2400 4200
+F 0 "D202" H 2400 4300 50  0000 C CNN
+F 1 "LED" H 2400 4100 50  0000 C CNN
+F 2 "" H 2400 4200 60  0001 C CNN
+F 3 "" H 2400 4200 60  0001 C CNN
+	1    2400 4200
 	0    -1   1    0
 $EndComp
@@
 Text HLabel 10650 3600 2    60   Output ~ 0
 M-
-Text HLabel 6900 2750 2    60   Input ~ 0
+Text HLabel 6900 3050 2    60   Input ~ 0
 aPot
-Text HLabel 6900 4550 2    60   Output ~ 0
+Text HLabel 6950 4550 2    60   Output ~ 0
 ISP_MISO
-Text HLabel 6900 4650 2    60   Input ~ 0
+Text HLabel 6950 4650 2    60   Input ~ 0
 ISP_MOSI
-Text HLabel 6900 4750 2    60   Input ~ 0
+Text HLabel 6950 4750 2    60   Input ~ 0
 ISP_SCK
 Text HLabel 4600 6200 2    60   BiDi ~ 0
@@
 L R R203
 U 1 1 50B6499F
-P 2000 4200
-F 0 "R203" V 2080 4200 50  0000 C CNN
-F 1 "400" V 2000 4200 50  0000 C CNN
-F 2 "" H 2000 4200 60  0001 C CNN
-F 3 "" H 2000 4200 60  0001 C CNN
-	1    2000 4200
+P 2000 3550
+F 0 "R203" V 2080 3550 50  0000 C CNN
+F 1 "400" V 2000 3550 50  0000 C CNN
+F 2 "" H 2000 3550 60  0001 C CNN
+F 3 "" H 2000 3550 60  0001 C CNN
+	1    2000 3550
 	1    0    0    -1
 $EndComp
@@
 L R R204
 U 1 1 50B649A5
-P 2400 4200
-F 0 "R204" V 2480 4200 50  0000 C CNN
-F 1 "400" V 2400 4200 50  0000 C CNN
-F 2 "" H 2400 4200 60  0001 C CNN
-F 3 "" H 2400 4200 60  0001 C CNN
-	1    2400 4200
-	1    0    0    -1
-$EndComp
-Wire Wire Line
-	2000 4450 2000 4550
+P 2400 3550
+F 0 "R204" V 2480 3550 50  0000 C CNN
+F 1 "400" V 2400 3550 50  0000 C CNN
+F 2 "" H 2400 3550 60  0001 C CNN
+F 3 "" H 2400 3550 60  0001 C CNN
+	1    2400 3550
+	1    0    0    -1
+$EndComp
+Wire Wire Line
+	2000 4400 2000 4550
 Wire Wire Line
 	2000 4550 2400 4550
 Wire Wire Line
-	2400 4550 2400 4450
+	2400 4550 2400 4400
 Wire Wire Line
 	2200 4650 2200 4550
@@
 Isense
 Wire Wire Line
-	6350 3050 6900 3050
-Text Label 6900 3050 2    60   ~ 0
+	6350 3850 6900 3850
+Text Label 6900 3850 2    60   ~ 0
 Isense
 NoConn ~ 6350 4450
 NoConn ~ 6350 4350
-NoConn ~ 6350 3850
-NoConn ~ 6350 3950
 NoConn ~ 6350 3450
 NoConn ~ 6350 3250
@@
 Wire Wire Line
 	2500 7450 2500 7350
-NoConn ~ 6350 4050
-Wire Wire Line
-	2000 3700 2000 3950
-Wire Wire Line
-	2400 3950 2400 3700
+Wire Wire Line
+	2000 3800 2000 4000
+Wire Wire Line
+	2400 4000 2400 3800
 $Comp
 L DRV8833-QFN U203
@@
 Wire Wire Line
 	6600 5750 7050 5750
-NoConn ~ 6350 4850
-NoConn ~ 6350 4950
 $Comp
 L CRYSTAL-4pin X201
@@
 Text Label 10100 3250 1    60   ~ 0
 Vcp
+Text Label 10050 4100 0    60   ~ 0
+vInt
+Text Label 6950 5050 2    60   ~ 0
+m_FAULT
+Wire Wire Line
+	6350 5050 6950 5050
 $EndSCHEMATC
